Commit message: launch + params work

File: install/turtlebot3_description/share/turtlebot3_description/gazebo/burger.gazebo.xacro (robot description, xacro)
@@ -1 +1,174 @@
-/home/pederba/ros2_ws/src/turtlebot3/turtlebot3_description/gazebo/burger.gazebo.xacro
+<?xml version="1.0"?>
+<robot xmlns:xacro="http://ros.org/wiki/xacro">
+  <xacro:macro name="burger_gazebo" params="prefix">
+  <xacro:property name="laser_visual"  value="true"/>
+  <xacro:property name="imu_ang_vel_noise_mean" value="0.0" />
+  <xacro:property name="imu_ang_vel_noise_stddev" value="2e-4" />
+  <xacro:property name="imu_ang_vel_noise_bias_mean" value="0.0000075" />
+  <xacro:property name="imu_ang_vel_noise_bias_stddev" value="0.0000008" />
+  <xacro:property name="imu_lin_acc_noise_mean" value="0.0" />
+  <xacro:property name="imu_lin_acc_noise_stddev" value="1.7e-2" />
+  <xacro:property name="imu_lin_acc_noise_bias_mean" value="0.1" />
+  <xacro:property name="imu_lin_acc_noise_bias_stddev" value="0.001" />
+  <gazebo reference="${prefix}base_link">
+    <material>Gazebo/DarkGrey</material>
+  </gazebo>
+  <gazebo reference="${prefix}wheel_left_link">
+    <mu1>10000</mu1>
+    <mu2>10000</mu2>
+    <kp>500000.0</kp>
+    <kd>10.0</kd>
+    <minDepth>0.001</minDepth>
+    <maxVel>1.0</maxVel>
+    <fdir1>0 0 0</fdir1>
+    <material>Gazebo/FlatBlack</material>
+  </gazebo>
+  <gazebo reference="${prefix}wheel_right_link">
+    <mu1>10000</mu1>
+    <mu2>10000</mu2>
+    <kp>500000.0</kp>
+    <kd>10.0</kd>
+    <minDepth>0.001</minDepth>
+    <maxVel>1.0</maxVel>
+    <fdir1>0 0 0</fdir1>
+    <material>Gazebo/FlatBlack</material>
+  </gazebo>
+  <gazebo reference="${prefix}caster_back_link">
+    <mu1>0.0</mu1>
+    <mu2>0.0</mu2>
+    <kp>10000.0</kp>
+    <kd>1.0</kd>
+    <minDepth>0.001</minDepth>
+    <maxVel>1.0</maxVel>
+    <material>Gazebo/FlatBlack</material>
+  </gazebo>
+  <gazebo reference="${prefix}imu_link">
+    <material>Gazebo/Grey</material>
+    <sensor type="imu" name="imu">
+      <always_on>true</always_on>
+      <update_rate>100.0</update_rate>
+      <imu>
+        <angular_velocity>
+          <x>
+            <noise type="gaussian">
+              <mean>${imu_ang_vel_noise_mean}</mean>
+              <stddev>${imu_ang_vel_noise_stddev}</stddev>
+              <bias_mean>${imu_ang_vel_noise_bias_mean}</bias_mean>
+              <bias_stddev>${imu_ang_vel_noise_bias_stddev}</bias_stddev>
+            </noise>
+          </x>
+          <y>
+            <noise type="gaussian">
+              <mean>${imu_ang_vel_noise_mean}</mean>
+              <stddev>${imu_ang_vel_noise_stddev}</stddev>
+              <bias_mean>${imu_ang_vel_noise_bias_mean}</bias_mean>
+              <bias_stddev>${imu_ang_vel_noise_bias_stddev}</bias_stddev>
+            </noise>
+          </y>
+          <z>
+            <noise type="gaussian">
+              <mean>${imu_ang_vel_noise_mean}</mean>
+              <stddev>${imu_ang_vel_noise_stddev}</stddev>
+              <bias_mean>${imu_ang_vel_noise_bias_mean}</bias_mean>
+              <bias_stddev>${imu_ang_vel_noise_bias_stddev}</bias_stddev>
+            </noise>
+          </z>
+        </angular_velocity>
+        <linear_acceleration>
+          <x>
+            <noise type="gaussian">
+              <mean>${imu_lin_acc_noise_mean}</mean>
+              <stddev>${imu_lin_acc_noise_stddev}</stddev>
+              <bias_mean>${imu_lin_acc_noise_bias_mean}</bias_mean>
+              <bias_stddev>${imu_lin_acc_noise_bias_stddev}</bias_stddev>
+            </noise>
+          </x>
+          <y>
+            <noise type="gaussian">
+              <mean>${imu_lin_acc_noise_mean}</mean>
+              <stddev>${imu_lin_acc_noise_stddev}</stddev>
+              <bias_mean>${imu_lin_acc_noise_bias_mean}</bias_mean>
+              <bias_stddev>${imu_lin_acc_noise_bias_stddev}</bias_stddev>
+            </noise>
+          </y>
+          <z>
+            <noise type="gaussian">
+              <mean>${imu_lin_acc_noise_mean}</mean>
+              <stddev>${imu_lin_acc_noise_stddev}</stddev>
+              <bias_mean>${imu_lin_acc_noise_bias_mean}</bias_mean>
+              <bias_stddev>${imu_lin_acc_noise_bias_stddev}</bias_stddev>
+            </noise>
+          </z>
+        </linear_acceleration>
+      </imu>
+    </sensor>
+  </gazebo>
+  <!-- <gazebo>
+    <plugin name='diff_drive' filename='libgazebo_ros_diff_drive.so'>
+      <ros>
+        <namespace></namespace>
+        <remapping>cmd_vel:=cmd_vel</remapping>
+        <remapping>odom:=odom</remapping>
+      </ros>
+      <left_joint>wheel_left_joint</left_joint>
+      <right_joint>wheel_right_joint</right_joint>
+      <wheel_separation>0.160</wheel_separation>
+      <wheel_diameter>0.066</wheel_diameter>
+      <max_wheel_torque>20</max_wheel_torque>
+      <max_wheel_acceleration>1.0</max_wheel_acceleration>
+      <publish_odom>true</publish_odom>
+      <publish_odom_tf>true</publish_odom_tf>
+      <publish_wheel_tf>false</publish_wheel_tf>
+      <odometry_frame>odom</odometry_frame>
+      <robot_base_frame>base_footprint</robot_base_frame>
+    </plugin>
+  </gazebo> -->
+  <gazebo>
+    <plugin name="gazebo_ros_p3d" filename="libgazebo_ros_p3d.so">
+        <ros>
+          <namespace>/</namespace>
+          <remapping>odom:=ground_truth</remapping>
+        </ros>
+        <body_name>base_footprint</body_name>
+        <frame_name>world</frame_name>
+        <update_rate>20</update_rate>
+      </plugin>
+  </gazebo>
+  <gazebo reference="${prefix}base_scan">
+    <material>Gazebo/FlatBlack</material>
+    <sensor type="ray" name="lds_lfcd_sensor">
+      <pose>0 0 0 0 0 0</pose>
+      <always_on>true</always_on>
+      <update_rate>5.0</update_rate>
+      <visualize>${laser_visual}</visualize>
+      <ray>
+        <scan>
+          <horizontal>
+            <samples>360</samples>
+            <resolution>1</resolution>
+            <min_angle>0.0</min_angle>
+            <max_angle>6.28319</max_angle>
+          </horizontal>
+        </scan>
+        <range>
+          <min>0.120</min>
+          <max>3.5</max>
+          <resolution>0.015</resolution>
+        </range>
+        <noise>
+          <type>gaussian</type>
+          <mean>0.0</mean>
+          <stddev>0.01</stddev>
+        </noise>
+      </ray>
+      <plugin name="gazebo_ros_lds_lfcd_controller" filename="libgazebo_ros_ray_sensor.so">
+        <ros>
+          <namespace></namespace>
+          <remapping>~/out:=scan</remapping>
+        </ros>
+        <output_type>sensor_msgs/LaserScan</output_type>
+      </plugin>
+    </sensor>
+  </gazebo>
+  </xacro:macro>
+</robot>

File: install/turtlebot3_description/share/turtlebot3_description/gazebo/materials.xacro (robot description, xacro)
@@ -1 +1,33 @@
-/home/pederba/ros2_ws/src/turtlebot3/turtlebot3_description/gazebo/materials.xacro
+<?xml version="1.0"?>
+<robot>
+  <material name="black">
+    <color rgba="0.0 0.0 0.0 1.0"/>
+  </material>
+  <material name="blue">
+    <color rgba="0.0 0.0 0.8 1.0"/>
+  </material>
+  <material name="brown">
+    <color rgba="0.8706 0.8118 0.7647 1.0"/>
+  </material>
+  <material name="dark">
+    <color rgba="0.3 0.3 0.3 1.0"/>
+  </material>
+  <material name="green">
+    <color rgba="0.0 0.8 0.0 1.0"/>
+  </material>
+  <material name="grey">
+    <color rgba="0.5 0.5 0.5 1.0"/>
+  </material>
+  <material name="light_black">
+    <color rgba="0.4 0.4 0.4 1.0"/>
+  </material>
+  <material name="orange">
+    <color rgba="1.0 0.4235 0.0392 1.0"/>
+  </material>
+  <material name="red">
+    <color rgba="0.8 0.0 0.0 1.0"/>
+  </material>
+  <material name="white">
+    <color rgba="1.0 1.0 1.0 1.0"/>
+  </material>
+</robot>

File: install/turtlebot3_description/share/turtlebot3_description/gazebo/waffle_pi.gazebo.xacro (robot description, xacro)
@@ -1 +1,159 @@
-/home/pederba/ros2_ws/src/turtlebot3/turtlebot3_description/gazebo/waffle_pi.gazebo.xacro
+<?xml version="1.0"?>
+<robot xmlns:xacro="http://ros.org/wiki/xacro">
+  <xacro:macro name="waffle_pi_gazebo" params="prefix">
+    <xacro:property name="laser_visual" value="true"/>
+    <xacro:property name="camera_visual" value="true"/>
+    <xacro:property name="imu_visual" value="true"/>
+    <gazebo reference="${prefix}base_link">
+      <material>Gazebo/DarkGrey</material>
+    </gazebo>
+    <gazebo reference="${prefix}wheel_left_link">
+      <mu1>10000</mu1>
+      <mu2>10000</mu2>
+      <kp>500000.0</kp>
+      <kd>10.0</kd>
+      <minDepth>0.001</minDepth>
+      <maxVel>0.1</maxVel>
+      <fdir1>1 0 0</fdir1>
+      <material>Gazebo/FlatBlack</material>
+    </gazebo>
+    <gazebo reference="${prefix}wheel_right_link">
+      <mu1>10000</mu1>
+      <mu2>10000</mu2>
+      <kp>500000.0</kp>
+      <kd>10.0</kd>
+      <minDepth>0.001</minDepth>
+      <maxVel>0.1</maxVel>
+      <fdir1>1 0 0</fdir1>
+      <material>Gazebo/FlatBlack</material>
+    </gazebo>
+    <gazebo reference="${prefix}caster_back_right_link">
+      <mu1>0.1</mu1>
+      <mu2>0.1</mu2>
+      <kp>1000000.0</kp>
+      <kd>100.0</kd>
+      <minDepth>0.001</minDepth>
+      <maxVel>1.0</maxVel>
+      <material>Gazebo/FlatBlack</material>
+    </gazebo>
+    <gazebo reference="${prefix}caster_back_left_link">
+      <mu1>0.1</mu1>
+      <mu2>0.1</mu2>
+      <kp>1000000.0</kp>
+      <kd>100.0</kd>
+      <minDepth>0.001</minDepth>
+      <maxVel>1.0</maxVel>
+      <material>Gazebo/FlatBlack</material>
+    </gazebo>
+    <gazebo reference="${prefix}imu_link">
+      <material>Gazebo/Grey</material>
+      <sensor type="imu" name="imu">
+        <always_on>true</always_on>
+        <update_rate>100.0</update_rate>
+        <visualize>${imu_visual}</visualize>
+      </sensor>
+    </gazebo>
+    <!-- <gazebo>
+    <plugin name='diff_drive' filename='libgazebo_ros_diff_drive.so'>
+      <ros>
+        <namespace></namespace>
+        <remapping>cmd_vel:=cmd_vel</remapping>
+        <remapping>odom:=odom</remapping>
+      </ros>
+      <left_joint>wheel_left_joint</left_joint>
+      <right_joint>wheel_right_joint</right_joint>
+      <wheel_separation>0.287</wheel_separation>
+      <wheel_diameter>0.066</wheel_diameter>
+      <max_wheel_torque>20</max_wheel_torque>
+      <max_wheel_acceleration>1.0</max_wheel_acceleration>
+      <publish_odom>true</publish_odom>
+      <publish_odom_tf>true</publish_odom_tf>
+      <publish_wheel_tf>false</publish_wheel_tf>
+      <odometry_frame>odom</odometry_frame>
+      <robot_base_frame>base_footprint</robot_base_frame>
+    </plugin>
+  </gazebo> -->
+    <gazebo>
+      <plugin name="gazebo_ros_p3d" filename="libgazebo_ros_p3d.so">
+        <ros>
+          <namespace></namespace>
+          <remapping>odom:=ground_truth</remapping>
+        </ros>
+        <body_name>base_footprint</body_name>
+        <frame_name>odom</frame_name>
+        <update_rate>20</update_rate>
+      </plugin>
+    </gazebo>
+    <gazebo reference="${prefix}base_scan">
+      <material>Gazebo/FlatBlack</material>
+      <sensor type="ray" name="lds_lfcd_sensor">
+        <pose>0 0 0 0 0 0</pose>
+        <always_on>true</always_on>
+        <update_rate>5.0</update_rate>
+        <visualize>${laser_visual}</visualize>
+        <ray>
+          <scan>
+            <horizontal>
+              <samples>360</samples>
+              <resolution>1</resolution>
+              <min_angle>0.0</min_angle>
+              <max_angle>6.28319</max_angle>
+            </horizontal>
+          </scan>
+          <range>
+            <min>0.120</min>
+            <max>3.5</max>
+            <resolution>0.015</resolution>
+          </range>
+          <noise>
+            <type>gaussian</type>
+            <mean>0.0</mean>
+            <stddev>0.01</stddev>
+          </noise>
+        </ray>
+        <plugin name="gazebo_ros_lds_lfcd_controller" filename="libgazebo_ros_ray_sensor.so">
+          <ros>
+            <namespace></namespace>
+            <remapping>~/out:=scan</remapping>
+          </ros>
+          <output_type>sensor_msgs/LaserScan</output_type>
+        </plugin>
+      </sensor>
+    </gazebo>
+    <gazebo reference="${prefix}camera_rgb_frame">
+      <sensor type="depth" name="pi_camera">
+        <update_rate>30</update_rate>
+        <always_on>true</always_on>
+        <visualize>${camera_visual}</visualize>
+        <camera>
+          <horizontal_fov>1.085595</horizontal_fov>
+          <image>
+            <width>640</width>
+            <height>480</height>
+            <format>R8G8B8</format>
+          </image>
+          <clip>
+            <near>0.03</near>
+            <far>100</far>
+          </clip>
+          <noise>
+            <type>gaussian</type>
+            <!-- Noise is sampled independently per pixel on each frame.
+                 That pixel's noise value is added to each of its color
+                 channels, which at that point lie in the range [0,1]. -->
+            <mean>0.0</mean>
+            <stddev>0.007</stddev>
+          </noise>
+        </camera>
+        <plugin name="camera_controller" filename="libgazebo_ros_camera.so">
+          <frame_name>camera_rgb_optical_frame</frame_name>
+          <ros>
+            <namespace></namespace>
+            <remapping>image_raw:=image_raw</remapping>
+            <remapping>camera_info:=camera_info</remapping>
+          </ros>
+        </plugin>
+      </sensor>
+    </gazebo>
+  </xacro:macro>
+</robot>

File: install/turtlebot3_description/share/turtlebot3_description/ros2_control/turtlebot3_system.ros2_control.xacro (robot description, xacro)
@@ -1 +1,101 @@
-/home/pederba/ros2_ws/src/turtlebot3/turtlebot3_description/ros2_control/turtlebot3_system.ros2_control.xacro
+<?xml version="1.0"?>
+<!--
+Copied and modified from ros2 control demos example:
+https://github.com/ros-controls/ros2_control_demos/blob/foxy/ros2_control_demo_description/diffbot_description/ros2_control/diffbot_system.ros2_control.xacro
+-->
+<robot xmlns:xacro="http://www.ros.org/wiki/xacro">
+  <xacro:macro name="turtlebot3_system" params="name prefix use_sim:=^|false use_fake_hardware:=^|false fake_sensor_commands:=^|false">
+    <ros2_control name="${name}" type="system">
+      <xacro:if value="$(arg use_sim)">
+        <hardware>
+          <plugin>gazebo_ros2_control/GazeboSystem</plugin>
+        </hardware>
+      </xacro:if>
+      <xacro:unless value="$(arg use_sim)">
+        <hardware>
+          <xacro:if value="${use_fake_hardware}">
+            <plugin>fake_components/GenericSystem</plugin>
+            <param name="fake_sensor_commands">${fake_sensor_commands}</param>
+            <param name="state_following_offset">0.0</param>
+          </xacro:if>
+          <xacro:unless value="${use_fake_hardware}">
+            <plugin>turtlebot3_hardware/TurtleBot3SystemHardware</plugin>
+            <param name="opencr_id">200</param>
+            <param name="opencr_usb_port">/dev/ttyACM0</param>
+            <param name="opencr_baud_rate">1000000</param>
+          </xacro:unless>
+        </hardware>
+      </xacro:unless>
+      <joint name="${prefix}wheel_left_joint">
+        <command_interface name="velocity">
+          <param name="min">-24.5</param>
+          <param name="max">24.5</param>
+        </command_interface>
+        <state_interface name="position">
+          <param name="initial_value">0.0</param>
+        </state_interface>
+        <state_interface name="velocity">
+          <param name="initial_value">0.0</param>
+        </state_interface>
+      </joint>
+      <joint name="${prefix}wheel_right_joint">
+        <command_interface name="velocity">
+          <param name="min">-24.5</param>
+          <param name="max">24.5</param>
+        </command_interface>
+        <state_interface name="position">
+          <param name="initial_value">0.0</param>
+        </state_interface>
+        <state_interface name="velocity">
+          <param name="initial_value">0.0</param>
+        </state_interface>
+      </joint>
+      <sensor name="imu">
+        <state_interface name="orientation.x">
+          <param name="initial_value">0.0</param>
+        </state_interface>
+        <state_interface name="orientation.y">
+          <param name="initial_value">0.0</param>
+        </state_interface>
+        <state_interface name="orientation.z">
+          <param name="initial_value">0.0</param>
+        </state_interface>
+        <state_interface name="orientation.w">
+          <param name="initial_value">0.0</param>
+        </state_interface>
+        <state_interface name="angular_velocity.x">
+          <param name="initial_value">0.0</param>
+        </state_interface>
+        <state_interface name="angular_velocity.y">
+          <param name="initial_value">0.0</param>
+        </state_interface>
+        <state_interface name="angular_velocity.z">
+          <param name="initial_value">0.0</param>
+        </state_interface>
+        <state_interface name="linear_acceleration.x">
+          <param name="initial_value">0.0</param>
+        </state_interface>
+        <state_interface name="linear_acceleration.y">
+          <param name="initial_value">0.0</param>
+        </state_interface>
+        <state_interface name="linear_acceleration.z">
+          <param name="initial_value">0.0</param>
+        </state_interface>
+      </sensor>
+      <sensor name="battery">
+        <state_interface name="voltage">
+          <param name="initial_value">0.0</param>
+        </state_interface>
+        <state_interface name="percentage">
+          <param name="initial_value">0.0</param>
+        </state_interface>
+        <state_interface name="design_capacity">
+          <param name="initial_value">0.0</param>
+        </state_interface>
+        <state_interface name="present">
+          <param name="initial_value">0.0</param>
+        </state_interface>
+      </sensor>
+    </ros2_control>
+  </xacro:macro>
+</robot>

File: install/turtlebot3_description/share/turtlebot3_description/urdf/burger.urdf.xacro (robot description, xacro)
@@ -1 +1,146 @@
-/home/pederba/ros2_ws/src/turtlebot3/turtlebot3_description/urdf/burger.urdf.xacro
+<?xml version="1.0"?>
+<!-- TurtleBot3 Burger -->
+<robot xmlns:xacro="http://www.ros.org/wiki/xacro">
+  <xacro:macro name="burger" params="prefix">
+  <xacro:property
+    name="meshes_file_direction"
+    value="package://turtlebot3_description/meshes/burger"/>
+  <link name="${prefix}base_footprint"/>
+  <joint name="${prefix}base_joint" type="fixed">
+    <parent link="${prefix}base_footprint"/>
+    <child link="${prefix}base_link" />
+    <origin xyz="0 0 0.010" rpy="0 0 0"/>
+  </joint>
+  <link name="${prefix}base_link">
+    <visual>
+      <origin xyz="-0.032 0 0.0" rpy="0 0 0"/>
+      <geometry>
+        <mesh filename="${meshes_file_direction}/base.stl" scale="0.001 0.001 0.001"/>
+      </geometry>
+      <material name="light_black"/>
+    </visual>
+    <collision>
+      <origin xyz="-0.032 0 0.070" rpy="0 0 0"/>
+      <geometry>
+        <box size="0.140 0.140 0.143"/>
+      </geometry>
+    </collision>
+    <inertial>
+      <origin xyz="0 0 0" rpy="0 0 0"/>
+      <mass value="8.2573504e-01"/>
+      <inertia ixx="2.2124416e-03" ixy="-1.2294101e-05" ixz="3.4938785e-05"
+               iyy="2.1193702e-03" iyz="-5.0120904e-06"
+               izz="2.0064271e-03" />
+    </inertial>
+  </link>
+  <joint name="${prefix}wheel_left_joint" type="continuous">
+    <parent link="${prefix}base_link"/>
+    <child link="${prefix}wheel_left_link"/>
+    <origin xyz="0.0 0.08 0.023" rpy="-1.57079632679 0 0"/>
+    <axis xyz="0 0 1"/>
+  </joint>
+  <link name="${prefix}wheel_left_link">
+    <visual>
+      <origin xyz="0 0 0" rpy="1.57079632679 0 0"/>
+      <geometry>
+        <mesh filename="${meshes_file_direction}/left_tire.stl" scale="0.001 0.001 0.001"/>
+      </geometry>
+      <material name="dark"/>
+    </visual>
+    <collision>
+      <origin xyz="0 0 0" rpy="0 0 0"/>
+      <geometry>
+        <cylinder length="0.018" radius="0.033"/>
+      </geometry>
+    </collision>
+    <inertial>
+      <origin xyz="0 0 0" />
+      <mass value="2.8498940e-02" />
+      <inertia ixx="1.1175580e-05" ixy="-4.2369783e-11" ixz="-5.9381719e-09"
+               iyy="1.1192413e-05" iyz="-1.4400107e-11"
+               izz="2.0712558e-05" />
+    </inertial>
+  </link>
+  <joint name="${prefix}wheel_right_joint" type="continuous">
+    <parent link="${prefix}base_link"/>
+    <child link="${prefix}wheel_right_link"/>
+    <origin xyz="0.0 -0.080 0.023" rpy="-1.57079632679 0 0"/>
+    <axis xyz="0 0 1"/>
+  </joint>
+  <link name="${prefix}wheel_right_link">
+    <visual>
+      <origin xyz="0 0 0" rpy="1.57079632679 0 0"/>
+      <geometry>
+        <mesh filename="${meshes_file_direction}/right_tire.stl" scale="0.001 0.001 0.001"/>
+      </geometry>
+      <material name="dark"/>
+    </visual>
+    <collision>
+      <origin xyz="0 0 0" rpy="0 0 0"/>
+      <geometry>
+        <cylinder length="0.018" radius="0.033"/>
+      </geometry>
+    </collision>
+    <inertial>
+      <origin xyz="0 0 0" />
+      <mass value="2.8498940e-02" />
+      <inertia ixx="1.1175580e-05" ixy="-4.2369783e-11" ixz="-5.9381719e-09"
+               iyy="1.1192413e-05" iyz="-1.4400107e-11"
+               izz="2.0712558e-05" />
+    </inertial>
+  </link>
+  <joint name="${prefix}caster_back_joint" type="fixed">
+    <parent link="${prefix}base_link"/>
+    <child link="${prefix}caster_back_link"/>
+    <origin xyz="-0.081 0 -0.004" rpy="-1.57079632679 0 0"/>
+  </joint>
+  <link name="${prefix}caster_back_link">
+    <collision>
+      <origin xyz="0 0 0" rpy="0 0 0"/>
+      <geometry>
+        <box size="0.030 0.009 0.020"/>
+      </geometry>
+    </collision>
+    <inertial>
+      <origin xyz="0 0 0" />
+      <mass value="0.005" />
+      <inertia ixx="0.001" ixy="0.0" ixz="0.0"
+               iyy="0.001" iyz="0.0"
+               izz="0.001" />
+    </inertial>
+  </link>
+  <joint name="${prefix}imu_joint" type="fixed">
+    <parent link="${prefix}base_link"/>
+    <child link="${prefix}imu_link"/>
+    <origin xyz="-0.032 0 0.068" rpy="0 0 0"/>
+  </joint>
+  <link name="${prefix}imu_link"/>
+  <joint name="${prefix}scan_joint" type="fixed">
+    <parent link="${prefix}base_link"/>
+    <child link="${prefix}base_scan"/>
+    <origin xyz="-0.032 0 0.172" rpy="0 0 0"/>
+  </joint>
+  <link name="${prefix}base_scan">
+    <visual>
+      <origin xyz="0 0 0.0" rpy="0 0 0"/>
+      <geometry>
+        <mesh filename="${meshes_file_direction}/ladar.stl" scale="0.001 0.001 0.001"/>
+      </geometry>
+      <material name="dark"/>
+    </visual>
+    <collision>
+      <origin xyz="0.015 0 -0.0065" rpy="0 0 0"/>
+      <geometry>
+        <cylinder length="0.0315" radius="0.055"/>
+      </geometry>
+    </collision>
+    <inertial>
+      <mass value="0.114" />
+      <origin xyz="0 0 0" />
+      <inertia ixx="0.001" ixy="0.0" ixz="0.0"
+               iyy="0.001" iyz="0.0"
+               izz="0.001" />
+    </inertial>
+  </link>
+  </xacro:macro>
+</robot>
